Commit message: Add files via upload

File: src/my_robot/urdf/my_robot.xacro (robot description, xacro)
@@ -180,3 +180,10 @@
     <axis xyz="0 1 0" rpy="0 0 0"/>
   </joint>
+  <joint name="camera_optical_joint" type="fixed">
+    <origin xyz="0 0 0" rpy="-1.5707 0 -1.5707"/>
+    <parent link="camera_link"/>
+    <child link="camera_link_optical"/>
+  </joint>
+  <link name="camera_link_optical">
+  </link>
 </robot>

Commit message: Add files via upload

File: src/my_robot/urdf/my_robot.xacro (robot description, xacro)
@@ -150,4 +150,11 @@
     <axis xyz="0 1 0" rpy="0 0 0"/>
   </joint>
+  <joint name="camera_optical_joint" type="fixed">
+    <origin xyz="0 0 0" rpy="-1.5707 0 -1.5707"/>
+    <parent link="camera"/>
+    <child link="camera_optical"/>
+  </joint>
+  <link name="camera_optical">
+  </link>
   <link name='hokuyo'>
     <pose>0 0 0.1 0 0 0</pose>
@@ -180,10 +187,3 @@
     <axis xyz="0 1 0" rpy="0 0 0"/>
   </joint>
-  <joint name="camera_optical_joint" type="fixed">
-    <origin xyz="0 0 0" rpy="-1.5707 0 -1.5707"/>
-    <parent link="camera"/>
-    <child link="camera_link_optical"/>
-  </joint>
-  <link name="camera_link_optical">
-  </link>
 </robot>
